Commit message: add terrain& rev02

File: assets/urdf/postech/urdf/postech.urdf (robot description, URDF)
Before this commit: robot postech, 7 links, 6 joints
Links:
- removed link leg_l_link
- removed link leg_r_link
- removed link shin_l_link
- removed link shin_r_link
- added link hip_l_link, mass 0.522076277648095; collision mesh filename=../meshes/hip_l_link.STL; visual mesh filename=../meshes/hip_l_link.STL
- added link hip_r_link, mass 0.522076277648095; collision mesh filename=../meshes/hip_r_link.STL; visual mesh filename=../meshes/hip_r_link.STL
- added link knee_l_link, mass 1.1404; collision mesh filename=../meshes/knee_l_link.STL; visual mesh filename=../meshes/knee_l_link.STL
- added link knee_r_link, mass 1.1404; collision mesh filename=../meshes/knee_r_link.STL; visual mesh filename=../meshes/knee_r_link.STL
Joints:
- removed joint leg_l_joint
- removed joint leg_r_joint
- removed joint shin_l_joint
- removed joint shin_r_joint
- added joint hip_l_joint: type revolute, parent base_link, child hip_l_link, origin xyz=-0.020921 0.212 -0.04807 rpy=-1.5708 0 0, axis 0 0 1, limit lower=-0.523599 upper=0.523599 effort=200 velocity=200
- added joint hip_r_joint: type revolute, parent base_link, child hip_r_link, origin xyz=-0.020921 -0.212 -0.04807 rpy=1.5708 0 0, axis 0 0 1, limit lower=-0.523599 upper=0.523599 effort=200 velocity=200
- added joint knee_l_joint: type revolute, parent hip_l_link, child knee_l_link, origin xyz=-0.18557 0.29001 0.0336 rpy=0 0 0, axis 0 0 1, limit lower=-0.20944 upper=0.959931 effort=200 velocity=200
- added joint knee_r_joint: type revolute, parent hip_r_link, child knee_r_link, origin xyz=-0.18557 -0.29001 0.0336 rpy=0 0 0, axis 0 0 1, limit lower=-0.20944 upper=0.959931 effort=200 velocity=200
- joint wheel_l_joint: limit effort=100 velocity=100 -> effort=1000 velocity=100; origin xyz=0.18657 0.29139 0.07725 rpy=0 0 0 -> xyz=0.18657 0.29139 0.0768 rpy=0 0 0; parent shin_l_link -> knee_l_link
- joint wheel_r_joint: limit effort=100 velocity=100 -> effort=1000 velocity=100; parent shin_r_link -> knee_r_link
