Commit message: updated obs buf

File: flamingo_env/assets/urdf/flamingo/urdf/flamingo.urdf (robot description, URDF)
Before this commit: robot flamingo, 9 links, 8 joints
Links:
- link base_link: mass 3.76040000 -> 4.00040000
- link right_hip_link: mass 0.92600000 -> 0.76800000
Joints:
- joint left_leg_joint: limit lower=0 upper=1.5708 effort=24 velocity=20 -> lower=-0.0872665 upper=1.5708 effort=24 velocity=20; origin xyz=0.17097 -0.13845 0.07005 rpy=0 0 0 -> xyz=0.22 0 0.07005 rpy=0 0 0
- joint left_shoulder_joint: limit lower=0 upper=1.5708 effort=24 velocity=20 -> lower=-0.785398 upper=0.785398 effort=24 velocity=20
- joint left_wheel_joint: origin xyz=-0.21779 0.031096 0.039877 rpy=0 0 0 -> xyz=-0.18883 -0.11289 0.039877 rpy=0 0 0
- joint right_leg_joint: limit lower=0 upper=1.5708 effort=24 velocity=20 -> lower=-0.0872665 upper=1.5708 effort=24 velocity=20; origin xyz=0.17097 0.13845 0.07005 rpy=0 0 0 -> xyz=0.22 0 0.07005 rpy=0 0 0
- joint right_shoulder_joint: limit lower=0 upper=1.5708 effort=24 velocity=20 -> lower=-0.785398 upper=0.785398 effort=24 velocity=20
- joint right_wheel_joint: origin xyz=-0.21779 -0.031096 0.039877 rpy=0 0 0 -> xyz=-0.18883 0.11289 0.039877 rpy=0 0 0

Commit message: wheel pos sin&cos added, action space added

File: flamingo_env/assets/urdf/flamingo/urdf/flamingo.urdf (robot description, URDF)
Before this commit: robot flamingo, 9 links, 8 joints
Joints:
- joint left_hip_joint: limit lower=-0.383972 upper=0.7854 effort=24 velocity=20 -> lower=-0.383972 upper=0.7854 effort=12 velocity=20
- joint left_leg_joint: limit lower=-0.0872665 upper=1.5708 effort=24 velocity=20 -> lower=-0.0872665 upper=1.5708 effort=12 velocity=20
- joint left_shoulder_joint: limit lower=-0.785398 upper=0.785398 effort=24 velocity=20 -> lower=-0.785398 upper=0.785398 effort=12 velocity=20
- joint left_wheel_joint: limit effort=6 velocity=50 -> effort=3 velocity=20
- joint right_hip_joint: limit lower=-0.7854 upper=0.383972 effort=24 velocity=20 -> lower=-0.7854 upper=0.383972 effort=12 velocity=20
- joint right_leg_joint: limit lower=-0.0872665 upper=1.5708 effort=24 velocity=20 -> lower=-0.0872665 upper=1.5708 effort=12 velocity=20
- joint right_shoulder_joint: limit lower=-0.785398 upper=0.785398 effort=24 velocity=20 -> lower=-0.785398 upper=0.785398 effort=12 velocity=20
- joint right_wheel_joint: limit effort=6 velocity=50 -> effort=3 velocity=20
